File: esp32.kicad_sch (KiCad schematic)
At the start: 27 parts, among them J1 USB_C_Receptacle, SW1 SW_SPST, SW2 SW_SPST, U1 ESP32-S3-WROOM-1, U3 AMS1117-3.3, U5 TPD2EUSB30A

Commit message: Reference board
Parts:
- removed C12: 10u, Capacitor_SMD:C_0805_2012Metric, symbol PCM_SparkFun-Capacitor:C
- removed C9: 0.1u, Capacitor_SMD:C_0603_1608Metric, symbol PCM_SparkFun-Capacitor:C
- added C3: 1u, Capacitor_SMD:C_0603_1608Metric, symbol PCM_SparkFun-Capacitor:C
- added C6: 100n, Capacitor_SMD:C_0805_2012Metric, symbol PCM_SparkFun-Capacitor:C
- added F1: 500mA, Fuse:Fuse_0603_1608Metric_Pad1.05x0.95mm_HandSolder, symbol Device:Fuse
- C7: value 0.1u -> 100n; Tolerance 10% -> 20%; Voltage 50V -> 25V
- renumbered C6 to C4, C10 to C5, C11 to C8, C8 to C9, D3 to D2, D2 to D3, R15 to R4, R11 to R5, R4 to R6, R14 to R7, U5 to U2, U2 to U4, U4 to U5
Connections:
- net +3V3: now also U5.19, F1.2; no longer C9.2, U3.2 (VO), U5.20
- net +5V: now also U5.20, C6.1; no longer C7.1, U5.19
- net CHIP_PU: now also C3.1
- net GND: now also C9.2, C3.2, C6.2; no longer C9.1
- net GPIO0: now also U5.10; no longer U5.13
- net GPIO14: now also U5.15; no longer U5.18
- net GPIO21: now also U5.14; no longer U5.17
- net GPIO45: now also U5.11; no longer U5.14
- net GPIO47: now also U5.13; no longer U5.16
- net GPIO48: now also U5.12; no longer U5.15
- net ESP_3V3 renamed +ESP_3V3
- net GPIO35: no longer names the net of U1.28 (IO35)
- net GPIO35: no longer U5.12
- net GPIO36: no longer names the net of U1.29 (IO36)
- net GPIO36: no longer U5.11
- net GPIO37: no longer names the net of U1.30 (IO37)
- net GPIO37: no longer U5.10
- net USB_DN renamed USB_D-
- net USB_DP renamed USB_D+
- new net 3V3_preFuse: C7.1, C9.1, F1.1, U3.2 (VO)
- no-connect marks 1 -> 7
Other:
- note added: "BUTTONS"
- note added: "PWR FLAGS"
- note added: "USB-C & LDO"
- note added: "USER LED"
- note removed: "LED"
- note removed: "USB-C"
- note removed: "Voltage Regulator LDO"
- moved on the sheet: C4, C5, C8, C9, D1, D2, D3, J1, R3, R4, R5, R6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
